Commit message: Fix duplicate gripper joint limit

File: urdf/arm.urdf.xacro (robot description, xacro)
@@ -182,5 +182,4 @@
     <origin xyz="-0.0275 0.057565 0.015" rpy="0 0 0"/>
     <axis xyz="0 0 1"/>
-    <limit lower="-0.50" upper="0.65" effort="10.0" velocity="2.0"/>
     <limit lower="0.00" upper="0.65" effort="10.0" velocity="2.0"/>
   </joint>
